File: Game_boy.kicad_pcb (KiCad board)
At the start: 2 copper layers, 130 x 51 mm, 61 parts, among them J1 USB_C_Receptacle_USB2.0_14P, J2 Conn_01x11, J3 Conn_01x04, SW1 SW_Push, SW2 SW_Push, SW3 SW_Push, SW4 SW_Push, SW5 SW_Push, SW6 SW_Push, SW7 SW_Push, SW8 SW_Push, SW9 SW_Push, U1 RT6154AGQW, U2 W25Q64JVXGIQ, U3 RP2040, Y1 12 MHz

Commit message: Update Readme
Parts:
- moved C1 94.1 mm to (82.5, 38.8)
- moved C13 94.1 mm to (80.3, 41.0)
- moved C19 94.1 mm to (103.7, 48.0)
- moved C2 94.1 mm to (86.5, 37.8)
- moved C4 94.1 mm to (74.3, 36.2)
- moved C5 94.1 mm to (90.9, 33.1)
- moved C8 94.1 mm to (81.5, 38.8)
- moved C9 94.1 mm to (85.5, 37.8)
- moved J2 94.1 mm to (115.9, 28.9)
- moved L1 94.1 mm to (71.4, 33.1)
- moved R1 94.1 mm to (92.5, 35.5)
- moved R10 94.1 mm to (84.5, 38.8)
- moved R11 94.1 mm to (83.5, 38.8)
- moved R3 94.1 mm to (92.5, 37.5)
- moved R4 94.1 mm to (86.9, 27.1)
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Routing:
- net GND: track 42.4 -> 44.5 mm

Commit message: First commit
Parts:
- removed the C7 at (75.5, 29.2)
- removed Card1: DM3AT-SF-PEJM5, easyeda2kicad:SD-SMD_DM3AT-SF-PEJM5
- removed the R5 at (80.0, 31.3)
- removed the R6 at (80.0, 30.3)
- removed TP3: TestPoint, TestPoint:TestPoint_Pad_1.0x1.0mm
- added C5: 22uF, Capacitor_SMD:C_1206_3216Metric, B.Cu at (77.2, 36.0)
- added R2: 100K, Resistor_SMD:R_0402_1005Metric, B.Cu at (76.3, 29.9)
- added R4: 1.02M, Resistor_SMD:R_0402_1005Metric, B.Cu at (76.1, 34.1)
- added TF1: TF-CARD H1.8, easyeda2kicad:TF-SMD_TF-CARD-H1.8, B.Cu at (104.0, 57.6)
- C4: value 47uF -> 10uF; footprint Capacitor_SMD:C_0805_2012Metric -> Capacitor_SMD:C_1206_3216Metric
- R7: value 1.02M -> 180K
- R8: value 180K -> 100K
- U1: value RT6154AGQW -> RT6150BGQW; footprint easyeda2kicad:VSON-14_L4.0-W3.0-P0.50-BL-EP_TI_DSJ -> easyeda2kicad:WSON-10_L2.5-W2.5-P0.50-BL-EP
- moved C4 8.91 mm to (77.7, 28.0), turned to 0 degrees
- moved TP1 7.15 mm to (75.3, 27.6)
- moved C20 6.92 mm to (106.7, 49.8), turned to -90 degrees
- moved TP2 5.26 mm to (74.5, 36.1)
- moved R8 4.98 mm to (79.4, 31.2), turned to 0 degrees
- moved C17 4.40 mm to (89.6, 55.0), turned to -90 degrees
- moved C19 2.43 mm to (105.0, 50.0)
- moved R15 2.43 mm to (109.4, 50.0)
- moved R16 2.43 mm to (108.3, 50.0)
- moved R17 2.43 mm to (103.9, 50.0)
- moved R18 2.43 mm to (102.8, 50.0)
- moved R19 2.43 mm to (101.7, 50.0)
- moved R7 2.42 mm to (78.2, 34.1)
- moved L1 1.51 mm to (72.4, 32.0)
- moved U1 1.10 mm to (76.5, 32.0), turned to 90 degrees
- renumbered C5 to C6, C6 to C7, R9 to R10, R2 to R3, R4 to R5, R3 to R6, R10 to R9
Connections:
- C4 pad 1: +3V3 -> VBUS
- L1 pad 1: Net-(L1-Pad1) -> Net-(U1-LX1)
- L1 pad 2: Net-(L1-Pad2) -> Net-(U1-LX2)
- R7 pad 1: +3V3 -> Net-(U1-FB)
- R7 pad 2: Net-(U1-FB) -> GND
- R8 pad 1: Net-(U1-FB) -> Net-(U1-PS)
- TP1 pad 1: +3V3 -> VBUS
- TP2 pad 1: VBUS -> +3V3
- U1 pad 1: VBUS -> +3V3
- U1 pad 10: VBUS -> Net-(U1-FB)
- U1 pad 11: VBUS -> GND
- U1 pad 2: GND -> Net-(U1-LX2)
- U1 pad 3: Net-(U1-FB) -> GND
- U1 pad 4: +3V3 -> Net-(U1-LX1)
- U1 pad 5: +3V3 -> VBUS
- U1 pad 6: Net-(L1-Pad2) -> Net-(U1-EN)
- U1 pad 7: Net-(L1-Pad2) -> Net-(U1-PS)
- U1 pad 8: Net-(L1-Pad1) -> VBUS
- U1 pad 9: Net-(L1-Pad1) -> GND
Routing:
- net +3V3: track 129.7 -> 143.8 mm, vias 6 -> 7
- net GND: track 44.5 -> 49.0 mm, vias 26 -> 22
- net Net-(L1-Pad2): track 4.17 -> 0.00 mm
- net Net-(L1-Pad1): track 4.14 -> 0.00 mm
- net RIGHT: track 70.8 -> 66.8 mm
- net VBUS: track 75.5 -> 71.6 mm, vias 3 -> 5
- net Net-(U1-PS/SYNC): track 3.22 -> 0.00 mm
- net Net-(U1-LX2): track 0.00 -> 3.15 mm
- net Net-(U1-LX1): track 0.00 -> 3.15 mm
- net Net-(U1-PGOOD): track 2.63 -> 0.00 mm, vias 1 -> 0
- net Net-(U1-EN): track 3.69 -> 1.32 mm
- net Net-(U1-FB): track 3.98 -> 2.22 mm
- net SD MISO: track 23.0 -> 24.5 mm
- net Net-(U1-PS): track 0.00 -> 1.43 mm
- net XIN: track 9.50 -> 10.4 mm
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- added copper zone on B.Cu, net +3V3
