File: Game_boy.kicad_sch (KiCad schematic)
At the start: 63 parts, among them J1 USB_C_Receptacle_USB2.0_14P, J2 Conn_01x11, J3 Conn_01x04, SW1 SW_Push, SW2 SW_Push, SW3 SW_Push, SW4 SW_Push, SW5 SW_Push, SW6 SW_Push, SW7 SW_Push, SW8 SW_Push, SW9 SW_Push, U1 RT6154AGQW, U2 W25Q64JVXGIQ, U3 RP2040, Y1 12 MHz

Commit message: Update Readme
Other:
- title: (none) -> Gameboy
- moved on the sheet: C1, C10, C11, C12, C13, C14, C15, C16, C17, C18, C19, C2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

Commit message: First commit
Parts:
- removed Card1: DM3AT-SF-PEJM5, easyeda2kicad:SD-SMD_DM3AT-SF-PEJM5, symbol SD-SMD_DM3AT-SF-PEJM5:DM3AT-SF-PEJM5
- removed TP3: TestPoint, TestPoint:TestPoint_Pad_1.0x1.0mm, symbol Connector:TestPoint
- removed U1: RT6154AGQW, easyeda2kicad:VSON-14_L4.0-W3.0-P0.50-BL-EP_TI_DSJ, symbol RT6154A:RT6154AGQW
- added TF1: TF-CARD H1.8, easyeda2kicad:TF-SMD_TF-CARD-H1.8, symbol TF-CARD H1.8:TF-CARDH1.8
- added U1: RT6150BGQW, easyeda2kicad:WSON-10_L2.5-W2.5-P0.50-BL-EP, symbol RT6150BGQW:RT6150BGQW
- C4: renamed from C7; value 47uF -> 10uF; footprint Capacitor_SMD:C_0805_2012Metric -> Capacitor_SMD:C_1206_3216Metric
- C5: renamed from C4; value 47uF -> 22uF; footprint Capacitor_SMD:C_0805_2012Metric -> Capacitor_SMD:C_1206_3216Metric
- renumbered C5 to C6, C6 to C7, R9 to R10, R6 to R2, R2 to R3, R7 to R4, R4 to R5, R3 to R6, R8 to R7, R5 to R8, R10 to R9, TP2 to TP1, TP1 to TP2
Connections:
- net +3V3: now also TF1.4 (VDD), U1.1 (VOUT)
- net GND: now also R8.2, TF1.10 (GND), TF1.11 (GND), TF1.12 (GND), TF1.13 (GND), TF1.6 (VSS), TF1.9 (CD), U1.11 (EXP), U1.3 (GND), U1.9 (GND)
- net SD CS: now also TF1.2 (CD/DAT3)
- net SD MISO: now also TF1.7 (DAT0)
- net SD MOSI: now also TF1.3 (CMD)
- net SD SCK: now also TF1.5 (CLK)
- net VBUS: now also U1.5 (VIN), U1.8 (VINA); no longer R8.1
- net at R4.2, R7.1: now also U1.10 (FB)
- net at R19.2: now also TF1.1 (DAT2)
- net at R2.2: now also U1.6 (EN)
- net at L1.1: now also U1.4 (LX1)
- net at L1.2: now also U1.2 (LX2)
- net at R15.2: now also TF1.8 (DAT1)
- new net: R8.1, U1.7 (PS)
Other:
- moved on the sheet: C1, C10, C11, C12, C13, C14, C15, C16, C17, C18, C19, C2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
